File: edge-b/hardware/kicad_sailframes-b1.kicad_sch (KiCad schematic)
At the start: 72 parts, among them J2 JST_PH_BAT, J3 U.FL, J5 MICROSD, J8 BNO085_SOCKET, J9 HOSYOND_3.5_TFT, U1 LC29HEAMD, U2 TP4056, U3 MT3608, U4 ESP32_DEVKIT_V1

Commit message: B1 schematic: fix pull-up topology bugs + ERC clean
Schematic fixes:
- Redrew R21/R22 I2C pull-ups as parallel topology (was chained series,
  shorting V3V3 to I2C_SDA/SCL)
- Redrew R23-R27 SD pull-ups as parallel topology (was chained series,
  shorting V3V3 to HSPI_CS/MOSI/MISO/SCK/SD_CD — would have destroyed
  the ESP32 once 3V3 hit GPIO5 through R23)
- Redrew C12-C16 V3V3 decap caps as parallel from V3V3 rail to GND
  (was chained, same merging issue)
- Changed TP4056 (U2) footprint from SOIC-8 to SOIC-8-1EP_3.9x4.9mm
  to expose pad 9 (thermal pad → GND)
- Deleted 2 dangling wire stubs near TP4056 and LATCH_Q_RB

ERC clean: 0 errors, 0 warnings. Cosmetic checks suppressed in project
settings (off-grid endpoints, Unspecified pin-type combinations, etc.).

PCB: F8 sync pulled in all 50 footprints; netlist now correct.

Co-Authored-By: Claude Opus 4.7 (1M context) <noreply@anthropic.com>
Parts:
- U2: footprint Package_SO:SOIC-8_3.9x4.9mm_P1.27mm -> Package_SO:SOIC-8-1EP_3.9x4.9mm_P1.27mm_EP2.29x3mm_ThermalVias
- renumbered J_QI to J_QI1, Q_INV to Q_INV1, Q_PWR to Q_PWR1, U_FF to U_FF1, U_HALL to U_HALL1, U_RST to U_RST1
Connections:
- net D2_ANODE: now also U2.7 (~{CHRG})
- net GNSS_RESET_N: no longer C10.1, L2.1, U1.9 (VDD_RF)
- net HSPI_CS: no longer C12.1, C13.1, C14.1, C15.1, C16.1, D10.2 (A), D11.1 (K), J5.2 (Pin_2), J5.3 (Pin_3), J5.4 (Pin_4), J5.5 (Pin_5), J8.1 (Pin_1), J8.4 (Pin_4), R16.1, R21.1, R21.2, R22.1, R23.1, R24.1, R24.2, R25.1, R25.2, R26.1, R26.2, R27.1, U1.23 (VCC), U4.11 (D14), U4.13 (D13), U4.16 (3V3), U4.26 (D21), U4.5 (D35)
- new net GNSS_VDD_RF: C10.1, L2.1, U1.9 (VDD_RF)
- new net HSPI_MISO: J5.3 (Pin_3), R25.2, U4.5 (D35)
- new net HSPI_MOSI: J5.2 (Pin_2), R24.2, U4.13 (D13)
- new net HSPI_SCK: J5.4 (Pin_4), R26.2, U4.11 (D14)
- new net I2C_SDA: J8.4 (Pin_4), R21.2, U4.26 (D21)
- new net V3V3: C12.1, C13.1, C14.1, C15.1, C16.1, D10.2 (A), D11.1 (K), J5.5 (Pin_5), J8.1 (Pin_1), R16.1, R21.1, R22.1, R23.1, R24.1, R25.1, R26.1, R27.1, U1.23 (VCC), U4.16 (3V3)
Other:
- moved on the sheet: C1, C10, C11, C12, C13, C14, C15, C16, C2, C3, C4, C5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
