File: edge-b/hardware/kicad_sailframes-b1.kicad_sch (KiCad schematic)
At the start: 78 parts, among them J10 I2C_EXP1, J11 I2C_EXP2, J12 I2C_EXP3, J13 GPIO_EXP, J14 UART_DBG, J15 J_AUX, J2 JST_PH_BAT, J3 U.FL, J5 MICROSD, J8 BNO085_SOCKET, J9 HOSYOND_3.5_TFT, U1 LC29HEAMD, U2 TP4056, U3 MT3608, U4 ESP32_DEVKIT_V1

Commit message: B1 schematic + project specs: add Hosyond TFT footprint, archive specs
B1 KiCad (kicad_sailframes-b1.kicad_sch + .kicad_pcb):
  * Add J9 = HOSYOND_3.5_TFT connector (1x10 2.54mm pin header,
    vertical) for the 3.5" 320x480 ST7796U IPS TFT module also used
    on the E-series enclosures
  * PCB layout + routing updates around the new connector

Project specs at repo root (now tracked):
  * B1_JAUX_HEADER_SPEC.md     — J_AUX expansion header spec
  * SF_FIRMWARE_V2_SPEC.md     — the v2.0.0 firmware roadmap that
    drove the .01 -> .09 Stage 1 work this session
  * SF_SHOPPING_LIST.md        — fleet hardware planning doc

Co-Authored-By: Claude Opus 4.7 (1M context) <noreply@anthropic.com>
Parts:
- J2: footprint Connector_JST:JST_PH_B2B-PH-K_1x02_P2.00mm_Vertical -> Connector_JST:JST_PH_S2B-PH-K_1x02_P2.00mm_Horizontal
- J9: footprint Connector_PinHeader_2.54mm:PinHeader_1x14_P2.54mm_Vertical -> Connector_PinHeader_2.54mm:PinHeader_1x10_P2.54mm_Vertical
Connections:
- net GND: now also J2.1 (Pin_1), J9.9 (GND); no longer J2.2 (Pin_2), J9.13 (GND)
- net TFT_BL: now also J9.3 (LED); no longer J9.7 (LED)
- net TFT_CS: now also J9.8 (LCD_CS); no longer J9.12 (LCD_CS)
- net TFT_DC: now also J9.6 (LCD_RS); no longer J9.10 (LCD_RS)
- net TFT_RST: now also J9.7 (LCD_RST); no longer J9.11 (LCD_RST)
- net V5_SW: now also J9.10 (VCC); no longer J9.14 (VCC)
- net VBAT: now also J2.2 (Pin_2); no longer J2.1 (Pin_1)
- net VSPI_MOSI: now also J9.5 (SDI_MOSI); no longer J9.9 (SDI_MOSI)
- net VSPI_SCK: now also J9.4 (SCK); no longer J9.8 (SCK)
- no-connect marks 26 -> 22
Other:
- moved on the sheet: D1, D4, D5, D6, R17, R18, R19, R20
