File: edge-b/hardware/kicad_sailframes-b1.kicad_sch (KiCad schematic)
At the start: 78 parts, among them J10 I2C_EXP1, J11 I2C_EXP2, J12 I2C_EXP3, J13 GPIO_EXP, J14 UART_DBG, J15 J_AUX, J2 JST_PH_BAT, J3 U.FL, J5 MICROSD, J8 BNO085_SOCKET, J9 HOSYOND_3.5_TFT, U1 LC29HEAMD, U2 TP4056, U3 MT3608, U4 ESP32_DEVKIT_V1

Commit message: B1 J_QI1: convert from THT connector to direct solder pads for Qi receiver wires
The Qi receiver module (coil + rectifier PCB) has 2 bare wire leads
(red V_QI / black GND). User decided to solder them directly into
plated through-holes on the B1 PCB rather than via a pin header.

PCB changes (J_QI1 footprint kept, geometry tweaked for wire soldering):
  - Pad 1 (V_QI):  1.7x1.7mm → 3.0x3.0mm,  drill 1.0 → 1.2mm
  - Pad 2 (GND):   1.7x1.7mm → 3.0x3.0mm,  drill 1.0 → 1.2mm
  - Pin spacing:   2.54mm → 4.0mm (better wire clearance)
  - Pad 1 stays rect (visual + polarity indicator for V_QI / red wire)
  - Pad 2 is circle
  - 1.2mm drill comfortably fits 22-24 AWG stripped wire with flux room
  - 3mm pads give good solder fillet for strain relief
  - Attribute marked: exclude_from_bom + dnp
    → JLCPCB will drill the holes but NOT install a connector

Schematic changes (J_QI1 symbol):
  - dnp: no → yes
  - in_bom: yes → no
  - in_pos_files: yes → no
  Symbol stays in schematic for documentation, but BOM and CPL
  exports will skip it.

Result: 2 plated through-holes (1.2mm diameter, 3mm pads, 4mm apart)
on F.Cu with no connector body. Hand-solder Qi receiver wires
directly into them after PCB arrives.
Parts:
- removed TP1: GNSS_TXD, TestPoint:TestPoint_Pad_1.0x1.0mm, symbol Connector:TestPoint
- removed TP2: GNSS_RXD, TestPoint:TestPoint_Pad_1.0x1.0mm, symbol Connector:TestPoint
- removed TP3: GNSS_RESET_N, TestPoint:TestPoint_Pad_1.0x1.0mm, symbol Connector:TestPoint
- removed TP4: GND, TestPoint:TestPoint_Pad_1.0x1.0mm, symbol Connector:TestPoint
- added J16: GNSS_DBG, Connector_PinHeader_2.54mm:PinHeader_1x04_P2.54mm_Vertical, symbol Connector_Generic:Conn_01x04
- added J17: LATCH_DBG, Connector_PinHeader_2.54mm:PinHeader_1x05_P2.54mm_Vertical, symbol Connector_Generic:Conn_01x05
- J_QI1: now not fitted; now left out of the parts list
Connections:
- net CLK_DEBOUNCED: now also J17.3 (Pin_3)
- net GND: now also J16.4 (Pin_4), J17.1 (Pin_1)
- net GNSS_RESET_N: now also J16.1 (Pin_1)
- net GNSS_RXD: now also J16.2 (Pin_2)
- net GNSS_TXD: now also J16.3 (Pin_3)
- net HALL_OUT: now also J17.2 (Pin_2)
- net LATCH_Q: now also J17.4 (Pin_4)
- net MOSFET_GATE: now also J17.5 (Pin_5)
- net EN: now reaches U4.1 (EN)
Other:
- moved on the sheet: C7, D10, D11, D8, J3, L1, Q_INV1, Q_PWR1, R14, R15, R16, R28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
