File: edge-b/hardware/kicad_sailframes-b1.kicad_sch (KiCad schematic)
At the start: 76 parts, among them J10 I2C_EXP1, J11 I2C_EXP2, J12 I2C_EXP3, J13 GPIO_EXP, J14 UART_DBG, J15 J_AUX, J16 GNSS_DBG, J17 LATCH_DBG, J2 JST_PH_BAT, J3 U.FL, J5 MICROSD, J8 BNO085_SOCKET, J9 HOSYOND_3.5_TFT, U1 LC29HEAMD, U2 TP4056, U3 MT3608, U4 ESP32_DEVKIT_V1

Commit message: B1 PCB: route board + DRC-clean, fix power/IMU bugs, add fab outputs
- Boost: fix inductor topology (L1 was out of the power path)
- D7 reversed to Option A (TP4056_VCC -> V5_SW); add C17 V_BCKP bypass
- J8 -> 10-pin GY-BNO08X pinout (3V3/GND/SCL/SDA), addr 0x4B
- Switcher re-placed tight; 4 mounting-hole keepouts (5.7mm)
- LED function silk (QI/CHRG/DONE/HB/GPS/SD); D/R refs moved to F.Fab
- Net classes (Power 0.5mm); fully routed, 0 DRC violations
- JLC fab package: gerbers, drill, BOM (bom-jlcpcb.csv), CPL

Co-Authored-By: Claude Opus 4.8 (1M context) <noreply@anthropic.com>
Parts:
- removed J8: BNO085_SOCKET, Connector_PinHeader_2.54mm:PinHeader_1x09_P2.54mm_Vertical, symbol Connector_Generic:Conn_01x09
- added C17: 100nF, Capacitor_SMD:C_0603_1608Metric, symbol Device:C
- added J1, J4: Conn_01x15, Connector_PinSocket_2.54mm:PinSocket_1x15_P2.54mm_Vertical, symbol Connector_Generic:Conn_01x15
- added J8: BNO085_DIRECT_SOLDER, Connector_PinHeader_2.54mm:PinHeader_1x10_P2.54mm_Vertical, symbol Connector_Generic:Conn_01x10
- C1, C13, C16, C3, C5, C9: LCSC Part # (none) -> C14663
- C10: LCSC Part # (none) -> C15195
- C11: LCSC Part # (none) -> C1546
- C12, C15, C2, C4, C7: LCSC Part # (none) -> C19702
- C14: LCSC Part # (none) -> C57112
- C8: LCSC Part # (none) -> C59461
- D1: LCSC Part # (none) -> C99290
- D10, D7, D8, D9: LCSC Part # (none) -> C2480
- D11: LCSC Part # (none) -> C7502694
- D2, D3: LCSC Part # (none) -> C125093
- D4: LCSC Part # (none) -> C2286
- D5: LCSC Part # (none) -> C2290
- J10, J11, J12, J13, J14, J15, J16, J17, J9: LCSC Part # (none) -> C2337
- J2: LCSC Part # (none) -> C173752
- J3: LCSC Part # (none) -> C88374
- J5: LCSC Part # (none) -> C719027
- J_QI1: footprint Connector_PinHeader_2.54mm:PinHeader_1x02_P2.54mm_Vertical -> Connector_Wire:SolderWire-0.5sqmm_1x02_P4.6mm_D0.9mm_OD2.1mm_Relief
- L1: LCSC Part # (none) -> C2044314
- L2: LCSC Part # (none) -> C32837
- Q_INV1: LCSC Part # (none) -> C20526
- Q_PWR1: LCSC Part # (none) -> C15127
- R1, R10, R12, R15, R2: LCSC Part # (none) -> C25803
- R11: LCSC Part # (none) -> C22793
- R13, R14, R16, R23, R24, R25, R26, R27, R28, R7: LCSC Part # (none) -> C15401
- R17, R18, R19: value 220 -> 1k; LCSC Part # (none) -> C21190
- R20: LCSC Part # (none) -> C23179
- R21, R22: LCSC Part # (none) -> C23162
- R6: LCSC Part # (none) -> C22975
- R8, R9: LCSC Part # (none) -> C21190
- U1: LCSC Part # (none) -> C28453488
- U2: LCSC Part # (none) -> C382139
- U3: LCSC Part # (none) -> C84817
- U4: now not fitted; now left out of the parts list
- U_FF1: footprint B1_JLC:SM8_L3.0-W2.8-P0.65-LS4.0-BL -> B1_JLC:VSSOP-8_DCU_2.3x2mm_P0.65mm; LCSC Part # (none) -> C70285
- U_HALL1: value DRV5032AJ -> DRV5032AJDBZR; footprint B1_DRV5032AJ:X2SON-4_L1.1-W1.4-P0.50-BR-EP -> Package_TO_SOT_SMD:SOT-23; LCSC Part # (none) -> C266120
- U_RST1: LCSC Part # (none) -> C347372
Connections:
- net BOOST_OUT is gone; now on net MT3608_SW: D9.2 (A), L1.2
- net AUX_INT: now also J1.2 (Pin_2)
- net D2_ANODE: no longer D2.1 (K), U2.7 (~{CHRG})
- net GND: now also C17.2, J1.14 (Pin_14), J4.2 (Pin_2), J8.2 (Pin_2); no longer U_HALL1.5 (EP)
- net GNSS_1PPS: now also J1.3 (Pin_3)
- net GNSS_RXD: now also J4.7 (Pin_7)
- net GNSS_TXD: now also J4.6 (Pin_6)
- net GNSS_V_BCKP: now also C17.1
- net GPIO12: now also J1.12 (Pin_12)
- net GPIO15: now also J4.3 (Pin_3)
- net HALL_OUT: now also U_HALL1.3 (OUT); no longer U_HALL1.4 (OUT)
- net HSPI_CS: now also J1.10 (Pin_10)
- net HSPI_MISO: now also J1.5 (Pin_5)
- net HSPI_MOSI: now also J1.13 (Pin_13)
- net HSPI_SCK: now also J1.11 (Pin_11)
- net I2C_SCL: now also J4.14 (Pin_14), J8.3 (Pin_3)
- net I2C_SDA: now also J4.11 (Pin_11), J8.4 (Pin_4)
- net LATCH_Q_RB: now also J4.10 (Pin_10)
- net LED_GPS_N: now also J1.6 (Pin_6)
- net LED_HB_N: now also J1.7 (Pin_7)
- net LED_SD_N: now also J1.9 (Pin_9)
- net MT3608_SW: no longer L1.1
- net RX0: now also J4.12 (Pin_12)
- net TFT_BL: now also J1.8 (Pin_8)
- net TFT_CS: now also J4.8 (Pin_8)
- net TFT_DC: now also J4.4 (Pin_4)
- net TFT_RST: now also J4.5 (Pin_5)
- net TP4056_VCC: now also D7.2 (A), R8.2, R9.2; no longer D7.1 (K)
- net TX0: now also J4.13 (Pin_13)
- net V3V3: now also J4.1 (Pin_1), J8.1 (Pin_1)
- net V5_SW: now also D7.1 (K), J1.15 (Pin_15); no longer D7.2 (A), R8.2, R9.2
- net VBAT: now also L1.1
- net VBAT_DIV: now also J1.4 (Pin_4)
- net VSPI_MOSI: now also J4.15 (Pin_15)
- net VSPI_SCK: now also J4.9 (Pin_9)
- net EN: no longer names the net of U4.1 (EN)
- new net TP_CHRG: D2.1 (K), U2.7 (~{CHRG})
- no-connect marks 22 -> 23
Other:
- moved on the sheet: C1, C2, C3, C4, C5, C9, D1, D2, D3, D4, D5, D6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
